File: Circuit/Kicad/V1/logic/logic/logic_p2.kicad_sch (KiCad schematic)
At the start: 2 parts

Commit message: LogicのPCBを途中まで作った
Parts:
- U1: renamed from U?; footprint (none) -> NUCLEO-STM32H7:NUCLEO-STM32H755ZI-Q
- U2: renamed from U?; footprint (none) -> RPI5:RPI5_GIPO
Connections:
- net D: now also U1.12 (PG14); no longer U1.13 (PG6)
- net E: now also U1.16 (PG8); no longer U1.12 (PG14)
Changed lines of the file:
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@@
     (stroke (width 0) (type default) (color 0 0 0 0))
   )
-  (wire (pts (xy 87.63 59.69) (xy 109.22 59.69))
+  (wire (pts (xy 101.6 120.65) (xy 101.6 118.11))
     (stroke (width 0) (type default) (color 0 0 0 0))
   )
@@
     (stroke (width 0) (type default) (color 0 0 0 0))
   )
+  (wire (pts (xy 110.49 125.73) (xy 99.06 125.73))
+    (stroke (width 0) (type default) (color 0 0 0 0))
+  )
   (wire (pts (xy 220.98 63.5) (xy 220.98 60.96))
     (stroke (width 0) (type default) (color 0 0 0 0))
   )
-  (wire (pts (xy 87.63 120.65) (xy 110.49 120.65))
-    (stroke (width 0) (type default) (color 0 0 0 0))
-  )
   (wire (pts (xy 194.31 66.04) (xy 220.98 66.04))
     (stroke (width 0) (type default) (color 0 0 0 0))
@@
     (stroke (width 0) (type default) (color 0 0 0 0))
   )
+  (wire (pts (xy 99.06 125.73) (xy 99.06 128.27))
+    (stroke (width 0) (type default) (color 0 0 0 0))
+  )
   (wire (pts (xy 87.63 123.19) (xy 110.49 123.19))
     (stroke (width 0) (type default) (color 0 0 0 0))
@@
     (stroke (width 0) (type default) (color 0 0 0 0))
   )
+  (wire (pts (xy 101.6 118.11) (xy 87.63 118.11))
+    (stroke (width 0) (type default) (color 0 0 0 0))
+  )
   (wire (pts (xy 194.31 86.36) (xy 220.98 86.36))
+    (stroke (width 0) (type default) (color 0 0 0 0))
+  )
+  (wire (pts (xy 110.49 120.65) (xy 101.6 120.65))
+    (stroke (width 0) (type default) (color 0 0 0 0))
+  )
+  (wire (pts (xy 99.06 128.27) (xy 87.63 128.27))
     (stroke (width 0) (type default) (color 0 0 0 0))
   )
@@
     (effects (font (size 1.27 1.27)) (justify left))
   )
-  (hierarchical_label "E" (shape output) (at 109.22 59.69 0)
+  (hierarchical_label "E" (shape output) (at 110.49 125.73 0)
     (effects (font (size 1.27 1.27)) (justify left))
   )
@@
   (symbol (lib_id "stm32h7:NUCLEO-H755ZI-Q_Zio") (at 77.47 36.83 0) (unit 1)
     (in_bom yes) (on_board yes) (fields_autoplaced)
-    (property "Reference" "U?" (id 0) (at 77.47 19.05 0)
+    (property "Reference" "U1" (id 0) (at 77.47 19.05 0)
       (effects (font (size 1.27 1.27)) hide)
     )
     (property "Value" "NUCLEO-H755ZI-Q_Zio" (id 1) (at 77.47 21.59 0))
-    (property "Footprint" "" (id 2) (at 90.17 26.67 0)
+    (property "Footprint" "NUCLEO-STM32H7:NUCLEO-STM32H755ZI-Q" (id 2) (at 90.17 26.67 0)
       (effects (font (size 1.27 1.27)) hide)
     )
@@
   (symbol (lib_id "power:+5V") (at 44.45 59.69 0) (unit 1)
     (in_bom yes) (on_board yes)
-    (property "Reference" "#PWR5V_2" (id 0) (at 44.45 52.07 0))
+    (property "Reference" "#PWR5V_06" (id 0) (at 44.45 52.07 0))
     (property "Value" "+5V" (id 1) (at 44.45 54.61 0))
     (property "Footprint" "" (id 2) (at 44.45 59.69 0)
@@
   (symbol (lib_id "power:GND") (at 220.98 72.39 0) (unit 1)
     (in_bom yes) (on_board yes) (fields_autoplaced)
-    (property "Reference" "#PWR?" (id 0) (at 220.98 78.74 0)
+    (property "Reference" "#PWR011" (id 0) (at 220.98 78.74 0)
       (effects (font (size 1.27 1.27)) hide)
     )
@@
   (symbol (lib_id "power:GND") (at 48.26 73.66 0) (unit 1)
     (in_bom yes) (on_board yes) (fields_autoplaced)
-    (property "Reference" "#PWR?" (id 0) (at 48.26 80.01 0)
+    (property "Reference" "#PWR010" (id 0) (at 48.26 80.01 0)
       (effects (font (size 1.27 1.27)) hide)
     )
@@
   (symbol (lib_id "rpi5:rpi5_GPIO") (at 179.07 58.42 0) (unit 1)
     (in_bom yes) (on_board yes) (fields_autoplaced)
-    (property "Reference" "U?" (id 0) (at 182.88 53.34 0)
+    (property "Reference" "U2" (id 0) (at 182.88 53.34 0)
       (effects (font (size 1.27 1.27)) hide)
     )
     (property "Value" "rpi5_GPIO" (id 1) (at 182.88 55.88 0))
-    (property "Footprint" "" (id 2) (at 179.07 58.42 0)
+    (property "Footprint" "RPI5:RPI5_GIPO" (id 2) (at 179.07 58.42 0)
       (effects (font (size 1.27 1.27)) hide)
     )
@@
   (symbol (lib_id "power:+5V") (at 220.98 55.88 0) (unit 1)
     (in_bom yes) (on_board yes)
-    (property "Reference" "#PWR5V_3" (id 0) (at 220.98 48.26 0))
+    (property "Reference" "#PWR5V_07" (id 0) (at 220.98 48.26 0))
     (property "Value" "+5V" (id 1) (at 220.98 50.8 0))
     (property "Footprint" "" (id 2) (at 220.98 55.88 0)
