File: Circuit/Kicad/V1/logic/logic/logic.kicad_pcb (KiCad board)
At the start: 2 copper layers, 51 parts, among them U1 NUCLEO-H755ZI-Q_Zio, U2 rpi5_GPIO

Commit message: can_transceiver周りのPCBを作った（仮）
Parts:
- moved REF2-2 135.2 mm to (147.3, 262.9)
- moved R4_TERM1 126.3 mm to (138.4, 265.4), turned to 90 degrees
- moved FB9 124.2 mm to (141.0, 273.1)
- moved FB10 124.1 mm to (141.0, 275.6)
- moved C18_Decupling1 122.6 mm to (138.4, 274.3), turned to 90 degrees
- moved C15_Decupling1 121.8 mm to (135.9, 262.9), turned to 90 degrees
- moved C14_Bypass1 121.5 mm to (133.6, 262.9), turned to -90 degrees
- moved C16_Bypass1 121.2 mm to (133.7, 274.3), turned to -90 degrees
- moved C17_Decupling1 120.9 mm to (137.2, 274.3), turned to 90 degrees
- moved Left_Leg1 117.8 mm to (127.0, 269.2)
- moved C12_Decupling1 115.3 mm to (116.8, 274.3), turned to 90 degrees
- moved C13_Bypass1 114.9 mm to (120.4, 274.3), turned to -90 degrees
- moved R2 114.4 mm to (116.8, 256.5)
- moved C11_Decupling1 114.1 mm to (115.6, 274.3), turned to 90 degrees
- moved FB6 112.9 mm to (113.0, 273.1)
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Connections:
- C1_Bypass1 pad : (no net) -> +5V
- C2_Decupling1 pad : (no net) -> +5V
- C3_Decupling1 pad : (no net) -> +5V
- C4_Bypass1 pad : (no net) -> GND
- C5_Bypass1 pad : (no net) -> +5V
- C6_Decupling1 pad : (no net) -> GND1
- C7_Bypass1 pad : (no net) -> GND1
- C8_Decupling1 pad : (no net) -> GND1
- C9_Decupling1 pad : (no net) -> +5V
- FB1 pad : (no net) -> +5V
- FB2 pad : (no net) -> GND
- FB3 pad : (no net) -> +5V
- FB4 pad : (no net) -> +5V
- FB5 pad : (no net) -> GND1
- R1 pad : (no net) -> +5V
- R2_TERM1 pad : (no net) -> CAN1_H
- REF1-2 pad 1: CAN1_H -> GND1 (x2)
- REF1-2 pad 2: CAN1_L -> CAN1_H (x2)
- REF1-2 pad 3: GND1 -> CAN1_L (x2)
- REF2-2 pad 1: CAN2_H -> GND1 (x2)
- REF2-2 pad 2: CAN2_L -> CAN2_H (x2)
- REF2-2 pad 3: GND1 -> CAN2_L (x2)
- Right-Leg1 pad 1: Net-(C1_Bypass1-Pad1) -> +5V
- Right-Leg1 pad 11: Net-(C7_Bypass1-Pad2) -> GND1
- Right-Leg1 pad 12: Net-(C7_Bypass1-Pad1) -> +5V
- Right-Leg1 pad 13: Net-(C7_Bypass1-Pad1) -> +5V
- Right-Leg1 pad 14: unconnected-(Right-Leg1-Pad14) -> GND1
- Right-Leg1 pad 2: /logic_p2/logic_p3/B -> /logic_p2/B
- Right-Leg1 pad 20: Net-(C5_Bypass1-Pad1) -> +5V
- Right-Leg1 pad 3: /logic_p2/logic_p3/CAN1_TX -> /logic_p2/CAN1_TX
- Right-Leg1 pad 4: /logic_p2/logic_p3/C -> /logic_p2/C
- Right-Leg1 pad 5: /logic_p2/logic_p3/CAN1_RX -> /logic_p2/CAN1_RX
- Right-Leg1 pad 7: unconnected-(Right-Leg1-Pad7) -> GND
- Right-Leg1 pad 9: Net-(C2_Decupling1-Pad1) -> +5V
Routing:
- net GND1: track 208.1 -> 293.5 mm, vias 0 -> 4
- net +5V: track 569.5 -> 637.6 mm
- net GND: track 415.7 -> 444.8 mm, vias 0 -> 2
- net /logic_p2/CAN1_RX: track 21.0 -> 38.4 mm, vias 0 -> 1
- net CAN1_H: track 0.00 -> 16.9 mm, vias 0 -> 3
- net /logic_p2/C: track 30.3 -> 47.1 mm, vias 0 -> 1
- net CAN1_L: track 0.00 -> 16.6 mm, vias 0 -> 3
- net /logic_p2/CAN1_TX: track 20.0 -> 36.3 mm, vias 0 -> 1
- net /logic_p2/B: track 22.6 -> 38.4 mm, vias 0 -> 1
- net Net-(R1-Pad1): track 0.00 -> 5.63 mm
- added copper zone on B.Cu, net GND
- added copper zone on F.Cu, net GND
- added copper zone on B.Cu, net GND1
- added copper zone on F.Cu, net GND1
Other:
- board text added: "Keep-out zone for any metal"
- board text added: "pin7(NC) -> GND pin14(GPIO output (default output is low)) -> GND これで良いのか？"
- board text added: "ここにDebug用のLEDつけたいね"

Commit message: can回路にLEDを追加。整理。
Parts:
- added D1: OSHR1608C1A, CAN_Pheripheral:OSHR1608C1A, F.Cu at (110.5, 233.7)
- added D2: OSHR1608C1A, CAN_Pheripheral:OSHR1608C1A, F.Cu at (143.5, 227.3)
- added R3: RK73B2ATTD121J, CAN_Pheripheral:RK73B2ATTD121J, F.Cu at (110.5, 229.9)
- added R4: RK73B2ATTD121J, CAN_Pheripheral:RK73B2ATTD121J, F.Cu at (143.5, 231.4)
- renumbered C1_Bypass1 to C1, C2_Decupling1 to C2, C3_Decupling1 to C3, C4_Bypass1 to C4, C5_Bypass1 to C5, C6_Decupling1 to C6, C7_Bypass1 to C7, C8_Decupling1 to C8, C9_Decupling1 to C9, R2_TERM1 to R2, R2 to R5, R4_TERM1 to R6_TERM1, Right-Leg1 to Right-Leg
Routing:
- net (no net): track 0.00 -> 4.39 mm
- net GND: track 444.8 -> 449.1 mm
- net +5V: track 637.6 -> 642.0 mm
- net GND1: track 293.5 -> 295.9 mm
Other:
- board outline added: 45.7 x 17.8 mm
- board text removed: "ここにDebug用のLEDつけたいね"

Commit message: スイッチの追加と整理。
Parts:
- removed REF**: AMASS_XT60-M_1x02_P7.20mm_Vertical, Connector_AMASS:AMASS_XT60-M_1x02_P7.20mm_Vertical
- added E-Button: AMASS_XT30U-M_1x02_P5.0mm_Vertical, Connector_AMASS:AMASS_XT30U-M_1x02_P5.0mm_Vertical, F.Cu at (22.9, 99.1)
- added Left_CAN: JST_XH_S2B-XH-A_1x02_P2.50mm_Horizontal, Connector_JST:JST_XH_S2B-XH-A_1x02_P2.50mm_Horizontal, F.Cu at (23.8, 130.8)
- added Logic_Supply: AMASS_XT60PW-M_1x02_P7.20mm_Horizontal, Connector_AMASS:AMASS_XT60PW-M_1x02_P7.20mm_Horizontal, F.Cu at (31.3, 121.7)
- added Power_GND: AMASS_XT30U-M_1x02_P5.0mm_Vertical, Connector_AMASS:AMASS_XT30U-M_1x02_P5.0mm_Vertical, F.Cu at (80.0, 162.6)
- added Q1: EKI04036, DCDC_Converter:EKI04036, F.Cu at (40.6, 109.2)
- added Q2: EKI04036, DCDC_Converter:EKI04036, F.Cu at (48.3, 109.2)
- added RPI_GPIO: RPI5_GIPO, RPI5:RPI5_GIPO, F.Cu at (81.3, 94.0)
- added RPI_SW: 2MS1-T1-B4-VS2-Q-E-S, DCDC_Converter:2MS1-T1-B4-VS2-Q-E-S, F.Cu at (48.3, 96.5)
- added Right_CAN: JST_XH_S2B-XH-A_1x02_P2.50mm_Horizontal, Connector_JST:JST_XH_S2B-XH-A_1x02_P2.50mm_Horizontal, F.Cu at (23.8, 160.0)
- added STM_SW: 2MS1-T1-B4-VS2-Q-E-S, DCDC_Converter:2MS1-T1-B4-VS2-Q-E-S, F.Cu at (41.9, 96.5)
- moved REF2-2 221.2 mm to (19.1, 152.4), turned to 180 degrees
- moved REF1-2 182.3 mm to (71.1, 152.4), turned to 180 degrees
- moved REF2-1 143.6 mm to (59.7, 152.4), turned to 180 degrees
- moved REF1-1 115.8 mm to (111.8, 152.4), turned to 180 degrees
- moved to_RPI1 19.9 mm to (90.2, 125.7)
- moved R_PU2 17.8 mm to (73.7, 121.7)
- moved R_PU1 17.7 mm to (73.7, 116.7)
- moved JET1 15.5 mm to (68.6, 101.6)
- moved for_PG1 15.5 mm to (59.7, 121.9)
- moved to_STM1 15.5 mm to (90.2, 108.0)
Connections:
- R_PU1 pad 2: Net-(R_PU1-Pad2) -> +5V
- R_PU2 pad 2: Net-(R_PU2-Pad2) -> +5V
- to_RPI1 pad 3: +5V -> GND
- to_STM1 pad 5: +12V -> GND
Routing:
- net +5V: track 642.0 -> 384.7 mm, vias 0 -> 2
- net /logic_p2/CAN2_RX: track 36.8 -> 191.0 mm, vias 0 -> 2
- net /logic_p2/D: track 15.8 -> 165.0 mm
- net /logic_p2/logic_p3/CAN2_TX: track 15.8 -> 162.4 mm
- net /logic_p2/E: track 15.8 -> 160.5 mm
- net /logic_p2/CAN1_TX: track 36.3 -> 140.8 mm, vias 1 -> 3
- net /logic_p2/CAN1_RX: track 38.4 -> 142.3 mm
- net /logic_p2/B: track 38.4 -> 138.8 mm, vias 1 -> 3
- net /logic_p2/C: track 47.1 -> 133.3 mm
- net GND: track 449.1 -> 373.0 mm, vias 2 -> 3
- net GND1: track 295.9 -> 224.9 mm
- net CAN1_L: track 16.6 -> 69.2 mm, vias 3 -> 4
- net CAN1_H: track 16.9 -> 69.5 mm, vias 3 -> 4
- net unconnected-(U1-Pad27): track 44.2 -> 0.00 mm
- net /logic_p2/A: track 30.5 -> 0.00 mm
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Other:
- board text added: "OFF"
- board text added: "ON"
- board text removed: "ココ、どう繋げる？コネクタを介す？"

Commit message: Version1のLogic基板が、形はできた。検査や見積もりはまだ
Parts:
- removed C10_Bypass1, C14_Bypass1: C_0.1uF, CAN_Pheripheral:GRM188F11H104ZA01
- removed C11_Decupling1, C15_Decupling1, C18_Decupling1: C_10uF, CAN_Pheripheral:GRM188R6YA106MA73
- removed C12_Decupling1, C17_Decupling1: C_1uF, CAN_Pheripheral:GRM188B31H105KAAL
- removed C13_Bypass1, C16_Bypass1: C_10nF, CAN_Pheripheral:GRM188B11H103KA01
- removed FB10, FB6, FB7, FB8, FB9: FerriteBead, CAN_Pheripheral:BLM21PG331SN
- removed Left_Leg1: ISOW1044, CAN_Transceiver:ISOW1044BDFMR
- removed R5: R_4.7k, CAN_Pheripheral:RK73B2ATTD472J
- removed R6_TERM1: R_120, CAN_Pheripheral:RK73B2ATTD121J
- removed the REF2-1 at (106.7, 262.9)
- removed the REF2-2 at (147.3, 262.9)
- added C1: C_0.1uF, CAN_Pheripheral:GRM188F11H104ZA01, F.Cu at (119.1, 179.1)
- added C2: C_10uF, CAN_Pheripheral:GRM188R6YA106MA73, F.Cu at (114.3, 189.2)
- added C3: C_1uF, CAN_Pheripheral:GRM188B31H105KAAL, F.Cu at (115.6, 189.2)
- added C4: C_10nF, CAN_Pheripheral:GRM188B11H103KA01, F.Cu at (119.1, 189.2)
- added C5: C_0.1uF, CAN_Pheripheral:GRM188F11H104ZA01, F.Cu at (132.3, 177.8)
- added C6: C_10uF, CAN_Pheripheral:GRM188R6YA106MA73, F.Cu at (134.6, 177.8)
- added C7: C_10nF, CAN_Pheripheral:GRM188B11H103KA01, F.Cu at (132.5, 189.2)
- added C8: C_1uF, CAN_Pheripheral:GRM188B31H105KAAL, F.Cu at (135.9, 189.2)
- added C9: C_10uF, CAN_Pheripheral:GRM188R6YA106MA73, F.Cu at (137.2, 189.2)
- added D1: OSHR1608C1A, CAN_Pheripheral:OSHR1608C1A, F.Cu at (109.2, 185.4)
- added D2: OSHR1608C1A, CAN_Pheripheral:OSHR1608C1A, F.Cu at (142.2, 179.1)
- added D_LED1: LED_D3.0mm, LED_THT:LED_D3.0mm, F.Cu at (115.5, 128.3)
- added D_LED2: LED_D3.0mm, LED_THT:LED_D3.0mm, F.Cu at (115.5, 110.5)
- added FB1: FerriteBead, CAN_Pheripheral:BLM21PG331SN, F.Cu at (111.8, 188.0)
- added FB2: FerriteBead, CAN_Pheripheral:BLM21PG331SN, F.Cu at (111.8, 190.5)
- added FB3: FerriteBead, CAN_Pheripheral:BLM21PG331SN, F.Cu at (114.3, 177.8)
- added FB4: FerriteBead, CAN_Pheripheral:BLM21PG331SN, F.Cu at (139.4, 188.0)
- added FB5: FerriteBead, CAN_Pheripheral:BLM21PG331SN, F.Cu at (139.4, 190.5)
- added Left-Leg: ISOW1044, CAN_Transceiver:ISOW1044BDFMR, F.Cu at (125.7, 184.2)
- added R1: R_4.7k, CAN_Pheripheral:RK73B2ATTD472J, F.Cu at (116.8, 182.9)
- added R2: R_120, CAN_Pheripheral:RK73B2ATTD121J, F.Cu at (137.2, 180.3)
- added R3: RK73B2ATTD102J, CAN_Pheripheral:RK73B2ATTD121J, F.Cu at (109.2, 181.6)
- added R4: RK73B2ATTD102J, CAN_Pheripheral:RK73B2ATTD121J, F.Cu at (142.2, 183.2)
- added REF**: MountingHole_3.2mm_M3, MountingHole:MountingHole_3.2mm_M3, F.Cu at (196.8, 24.1)
- added REF**: MountingHole_3.2mm_M3, MountingHole:MountingHole_3.2mm_M3, F.Cu at (25.4, 24.1)
- added REF**: MountingHole_3.2mm_M3, MountingHole:MountingHole_3.2mm_M3, F.Cu at (25.4, 166.4)
- added REF**: MountingHole_3.2mm_M3, MountingHole:MountingHole_3.2mm_M3, F.Cu at (196.8, 166.4)
- added REF1-1: PinHeader_1x06_P2.54mm_Vertical, Connector_PinHeader_2.54mm:PinHeader_1x06_P2.54mm_Vertical, F.Cu at (105.4, 177.8)
- added REF1-2: PinHeader_1x06_P2.54mm_Vertical, Connector_PinHeader_2.54mm:PinHeader_1x06_P2.54mm_Vertical, F.Cu at (146.1, 177.8)
- R3, R4: value RK73B2ATTD121J -> RK73B2ATTD102J
- moved C1 69.2 mm to (70.8, 179.1)
- moved C2 69.2 mm to (66.0, 189.2)
- moved C3 69.2 mm to (67.3, 189.2)
- moved C4 69.2 mm to (70.8, 189.2)
- moved C5 69.2 mm to (84.1, 177.8)
- moved C7 69.2 mm to (84.2, 189.2)
- moved C8 69.2 mm to (87.6, 189.2)
- moved C9 69.2 mm to (88.9, 189.2)
- moved D1 69.2 mm to (61.0, 185.4)
- moved D2 69.2 mm to (94.0, 179.1)
- moved FB1 69.2 mm to (63.5, 188.0)
- moved FB2 69.2 mm to (63.5, 190.5)
- moved R1 69.2 mm to (68.6, 182.9)
- moved R2 69.2 mm to (88.9, 180.3)
- moved R3 69.2 mm to (61.0, 181.6)
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- renumbered to_RPI1 to to_RPI, to_STM1 to to_STM
Connections:
- Power_GND pad 2: (no net) -> GND1
Routing:
- net +12V: track 203.0 -> 70.8 mm
- net +5V: track 384.7 -> 287.7 mm
- net GND1: track 224.9 -> 297.0 mm, vias 4 -> 8
- net GND: track 373.0 -> 411.7 mm, vias 3 -> 4
- net /logic_p2/CAN1_RX: track 142.3 -> 159.7 mm, vias 1 -> 2
- net CAN1_L: track 69.2 -> 86.3 mm, vias 4 -> 7
- net CAN1_H: track 69.5 -> 86.3 mm, vias 4 -> 7
- net /logic_p2/C: track 133.3 -> 150.2 mm, vias 1 -> 2
- net /logic_p2/CAN1_TX: track 140.8 -> 157.1 mm, vias 3 -> 4
- net /logic_p2/B: track 138.8 -> 154.6 mm, vias 3 -> 4
- net Net-(R1-Pad1): track 5.63 -> 11.3 mm
- net (no net): track 4.39 -> 8.78 mm
- added copper zone on F.Cu, net +12V
- added copper zone on F.Cu, net +5V
Other:
- board size 45.7 x 17.8 mm -> 184.1 x 175.3 mm
- board text removed: "GND1、どのように接続する？ XT90？ 基板用の端子台？ ねじ止めのハウジング？"
- board text removed: "Keep-out zone for any metal"
- board text removed: "pin7(NC) -> GND pin14(GPIO output (default output is low)) -> GND これで良いのか？"

Commit message: シルクを直した
Parts:
- renumbered REF2-2 to Left_CAN_Trans_Power, R_PU1 to R_PUp1, R_PU2 to R_PUp2, REF2-1 to Right_CAN_Trans_Logic, REF1-1 to Right_CAN_Trans_Logic, REF1-2 to Right_CAN_Trans_Power
Connections:
- C1 pad : +5V -> GND
- C2 pad : +5V -> GND
- C3 pad : +5V -> GND
- C8 pad : GND1 -> +5V
- C9 pad : +5V -> GND1
- R2 pad : CAN1_H -> CAN1_L
Other:
- board text added: "Left_Leg_Isolated_CAN_Transceiver"
- board text added: "NUCLEO SIM32 H755HZ"
- board text added: "Raspberry Pi 5"
- board text added: "Right_Leg_Isolated_CAN_Transceiver"

Commit message: v1-3ぐらい
Other:
- board text added: "NUCLEO-H755ZI-Q"
- board text removed: "NUCLEO SIM32 H755HZ"
Changed lines of the file:
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@@
   (gr_line (start 54.61 193.04) (end 54.61 175.26) (layer "Edge.Cuts") (width 0.1))
   (gr_line (start 102.87 193.04) (end 102.87 175.26) (layer "Edge.Cuts") (width 0.1))
-  (gr_text "NUCLEO SIM32 H755HZ" (at 156.21 161.29) (layer "F.SilkS")
+  (gr_text "NUCLEO-H755ZI-Q" (at 156.21 161.29) (layer "F.SilkS")
     (effects (font (size 1 1) (thickness 0.15)))
   )
@@
     (effects (font (size 1 1) (thickness 0.15)))
   )
+  (dimension (type aligned) (layer "F.SilkS")
+    (pts (xy 203.2 17.78) (xy 19.05 17.78))
+    (height 13.969999)
+    (gr_text "184.1500 mm" (at 111.125 -2.339999) (layer "F.SilkS")
+      (effects (font (size 6 6) (thickness 0.15)))
+    )
+    (format (units 3) (units_format 1) (precision 4))
+    (style (thickness 0.15) (arrow_length 1.27) (text_position_mode 0) (extension_height 0.58642) (extension_offset 0.5) keep_text_aligned)
+  )
+  (dimension (type aligned) (layer "F.SilkS")
+    (pts (xy 180.34 17.78) (xy 180.34 172.72))
+    (height -39.37)
+    (gr_text "154.9400 mm" (at 213.56 95.25 90) (layer "F.SilkS")
+      (effects (font (size 6 6) (thickness 0.15)))
+    )
+    (format (units 3) (units_format 1) (precision 4))
+    (style (thickness 0.15) (arrow_length 1.27) (text_position_mode 0) (extension_height 0.58642) (extension_offset 0.5) keep_text_aligned)
+  )
   (segment (start 60.96 182.61) (end 60.96 184.67) (width 0.6) (layer "F.Cu") (net 0))
