File: Circuit/Kicad/V2/RDC_Humanoid_Logic/CAN_Trans.kicad_sch (KiCad schematic)
At the start: 17 parts, among them U1 ISOW1044

Commit message: V2基板手直し
Connections:
- net GND2: no longer names the net of C3.2, C4.2, C5.2, FB1.2, U1.10 (GND1)
- net GND3: no longer names the net of C10.2, C11.2, C8.2, FB5.1, U1.11 (GND2)
Changed lines of the file:
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@@
-    (stroke (width 0) (type default))
-  )
-  (wire (pts (xy 190.5 114.3) (xy 190.5 124.46))
     (stroke (width 0) (type default))
   )
@@
   )
   (wire (pts (xy 190.5 114.3) (xy 190.5 109.22))
-    (stroke (width 0) (type default))
-  )
-  (wire (pts (xy 107.95 114.3) (xy 107.95 123.19))
     (stroke (width 0) (type default))
   )
@@
     )
   )
-  (symbol (lib_id "power:GND2") (at 107.95 123.19 0) (unit 1)
-    (in_bom yes) (on_board yes) (dnp no) (fields_autoplaced)
-    (property "Reference" "#PWR047" (at 107.95 129.54 0)
-      (effects (font (size 1.27 1.27)) hide)
-    )
-    (property "Value" "GND2" (at 107.95 128.27 0)
-      (effects (font (size 1.27 1.27)))
-    )
-    (property "Footprint" "" (at 107.95 123.19 0)
-      (effects (font (size 1.27 1.27)) hide)
-    )
-    (property "Datasheet" "" (at 107.95 123.19 0)
-      (effects (font (size 1.27 1.27)) hide)
-    )
-    (pin "1")
-    (instances
-      (project "RDC_Humanoid_Logic"
-        (path "/2bec3ac6-4176-417a-a2e5-e81844f01e63/2ffb334c-541d-4787-8f08-8f2b280267fd"
-          (reference "#PWR047") (unit 1)
-        )
-        (path "/2bec3ac6-4176-417a-a2e5-e81844f01e63/4e0cc178-8164-45af-8b1c-3daea8e76e2d"
-          (reference "#PWR048") (unit 1)
-        )
-      )
-    )
-  )
   (symbol (lib_id "power:GND") (at 90.17 123.19 0) (unit 1)
     (in_bom yes) (on_board yes) (dnp no) (fields_autoplaced)
@@
         )
       )
-    )
-  )
-  (symbol (lib_id "power:GND3") (at 190.5 124.46 0) (unit 1)
-    (in_bom yes) (on_board yes) (dnp no)
-    (property "Reference" "#PWR012" (at 190.5 130.81 0)
-      (effects (font (size 1.27 1.27)) hide)
-    )
-    (property "Value" "GND3" (at 190.5 128.27 0)
-      (effects (font (size 1.27 1.27)))
-    )
-    (property "Footprint" "" (at 190.5 124.46 0)
-      (effects (font (size 1.27 1.27)) hide)
-    )
-    (property "Datasheet" "" (at 190.5 124.46 0)
-      (effects (font (size 1.27 1.27)) hide)
-    )
-    (pin "1")
-    (instances
-      (project "RDC_Humanoid_Logic"
-        (path "/2bec3ac6-4176-417a-a2e5-e81844f01e63/2ffb334c-541d-4787-8f08-8f2b280267fd"
-          (reference "#PWR012") (unit 1)
-        )
-        (path "/2bec3ac6-4176-417a-a2e5-e81844f01e63/4e0cc178-8164-45af-8b1c-3daea8e76e2d"
-          (reference "#PWR016") (unit 1)
-        )
-      )

Commit message: 部品表の作成、多少のFootPrint、PCBの変更
Parts:
- R3, R4: footprint Resistor_SMD:R_0805_2012Metric -> Resistor_SMD:R_0603_1608Metric
Changed lines of the file:
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@@
       (effects (font (size 1.27 1.27)) (justify left))
     )
-    (property "Footprint" "Resistor_SMD:R_0805_2012Metric" (at 187.452 82.55 90)
+    (property "Footprint" "Resistor_SMD:R_0603_1608Metric" (at 187.452 82.55 90)
       (effects (font (size 1.27 1.27)) hide)
     )
@@
       (effects (font (size 1.27 1.27)) hide)
     )
-    (property "Datasheet" "" (at 144.78 78.74 0)
+    (property "Datasheet" "https://www.ti.com/lit/ds/symlink/isow1044.pdf?ts=1742141302334&ref_url=https%253A%252F%252Fwww.ti.com%252Fproduct%252Fja-jp%252FISOW1044%253Futm_source%253Dgoogle%2526utm_medium%253Dcpc%2526utm_campaign%253Depd-dlp-null-44700045336317809_prodfolderdynamic-cpc-pf-google-jp_jp_int%2526utm_content%253Dprodfolddynamic%2526ds_k%253DDYNAMIC+SEARCH+ADS%2526DCM%253Dyes%2526gclsrc%253Daw.ds%2526gad_source%253D1%2526gclid%253DCj0KCQjw7dm-BhCoARIsALFk4v-WAdcAF-zrUphoWc5iGoZEE4knVFtb3oJczRt-ALRTDiCCWS0eNeIaAqkBEALw_wcB" (at 144.78 78.74 0)
       (effects (font (size 1.27 1.27)) hide)
     )
@@
       (effects (font (size 1.27 1.27)) (justify left))
     )
-    (property "Footprint" "Resistor_SMD:R_0805_2012Metric" (at 112.268 74.93 90)
-      (effects (font (size 1.27 1.27)) hide)
-    )
+    (property "Footprint" "Resistor_SMD:R_0603_1608Metric" (at 112.268 74.93 90)
+      (effects (font (size 1.27 1.27)) hide)
+    )
