File: Circuit/Kicad/V2/RDC_Humanoid_Logic/RDC_Humanoid_Logic.kicad_pcb (KiCad board)
At the start: 2 copper layers, 157 x 137 mm, 70 parts, among them J1 XT60, J2 Conn_01x03, J3 Conn_01x03, J4 Raspi_connect, Q1 Q_PMOS_GDS, Q2 Q_PMOS_GDS, SW1 SW_SPDT, SW2 SW_SPDT, SW3 SW_SPDT, U1 ISOW1044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

Commit message: gbrの生成
Parts:
- moved C1 16.5 mm to (83.6, 59.4), turned to 0 degrees
Connections:
- C1 pad 1: +12V -> Logic_Power
Routing:
- net GND: vias 269 -> 270
Changed lines of the file:
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@@
       (drillshape 0)
       (scaleselection 1)
-      (outputdirectory "")
+      (outputdirectory "../Gerbers/Logic/")
     )
   )
@@
       (stroke (width 0.1) (type solid)) (layer "F.Fab"))
     (pad "" np_thru_hole oval (at 2.5 6.5) (size 2.8 2) (drill oval 2.8 2) (layers "*.Cu" "*.Mask"))
-    (pad "1" thru_hole roundrect (at 0 0) (size 1.7 1.95) (drill 0.95) (layers "*.Cu" "*.Mask") (roundrect_rratio 0.147059)
+    (pad "1" thru_hole roundrect (at 0 0) (size 1.7 1.95) (drill 0.95) (layers "*.Cu" "*.Mask") (roundrect_rratio 0.1470588235)
       (net 4 "GND1") (pinfunction "Pin_1") (pintype "passive"))
     (pad "2" thru_hole oval (at 2.5 0) (size 1.7 1.95) (drill 0.95) (layers "*.Cu" "*.Mask")
@@
     (fp_line (start 4.11 2.7) (end 3.11 2.7)
       (stroke (width 0.1) (type solid)) (layer "F.Fab"))
-    (pad "1" smd roundrect (at -5.04 -2.28 180) (size 2.2 1.2) (layers "F.Cu" "F.Paste" "F.Mask") (roundrect_rratio 0.208333)
+    (pad "1" smd roundrect (at -5.04 -2.28 180) (size 2.2 1.2) (layers "F.Cu" "F.Paste" "F.Mask") (roundrect_rratio 0.2083333333)
       (net 33 "Net-(Q1-G)") (pinfunction "G") (pintype "input"))
-    (pad "2" smd roundrect (at -0.415 -1.525 180) (size 3.05 2.75) (layers "F.Cu" "F.Paste") (roundrect_rratio 0.090909)
+    (pad "2" smd roundrect (at -0.415 -1.525 180) (size 3.05 2.75) (layers "F.Cu" "F.Paste") (roundrect_rratio 0.09090909091)
       (net 20 "Net-(Q1-D)") (pinfunction "D") (pintype "passive"))
-    (pad "2" smd roundrect (at -0.415 1.525 180) (size 3.05 2.75) (layers "F.Cu" "F.Paste") (roundrect_rratio 0.090909)
+    (pad "2" smd roundrect (at -0.415 1.525 180) (size 3.05 2.75) (layers "F.Cu" "F.Paste") (roundrect_rratio 0.09090909091)
       (net 20 "Net-(Q1-D)") (pinfunction "D") (pintype "passive"))
-    (pad "2" smd roundrect (at 1.26 0 180) (size 6.4 5.8) (layers "F.Cu" "F.Mask") (roundrect_rratio 0.043103)
+    (pad "2" smd roundrect (at 1.26 0 180) (size 6.4 5.8) (layers "F.Cu" "F.Mask") (roundrect_rratio 0.04310293103)
       (net 20 "Net-(Q1-D)") (pinfunction "D") (pintype "passive"))
-    (pad "2" smd roundrect (at 2.935 -1.525 180) (size 3.05 2.75) (layers "F.Cu" "F.Paste") (roundrect_rratio 0.090909)
+    (pad "2" smd roundrect (at 2.935 -1.525 180) (size 3.05 2.75) (layers "F.Cu" "F.Paste") (roundrect_rratio 0.09090909091)
       (net 20 "Net-(Q1-D)") (pinfunction "D") (pintype "passive"))
-    (pad "2" smd roundrect (at 2.935 1.525 180) (size 3.05 2.75) (layers "F.Cu" "F.Paste") (roundrect_rratio 0.090909)
+    (pad "2" smd roundrect (at 2.935 1.525 180) (size 3.05 2.75) (layers "F.Cu" "F.Paste") (roundrect_rratio 0.09090909091)
       (net 20 "Net-(Q1-D)") (pinfunction "D") (pintype "passive"))
-    (pad "3" smd roundrect (at -5.04 2.28 180) (size 2.2 1.2) (layers "F.Cu" "F.Paste" "F.Mask") (roundrect_rratio 0.208333)
+    (pad "3" smd roundrect (at -5.04 2.28 180) (size 2.2 1.2) (layers "F.Cu" "F.Paste" "F.Mask") (roundrect_rratio 0.2083333333)
       (net 168 "Logic_Power") (pinfunction "S") (pintype "passive"))
     (model "${KICAD6_3DMODEL_DIR}/Package_TO_SOT_SMD.3dshapes/TO-252-2.wrl"
@@
       (stroke (width 0.1) (type solid)) (layer "F.Fab"))
     (pad "" np_thru_hole oval (at 2.5 6.5) (size 2.8 2) (drill oval 2.8 2) (layers "*.Cu" "*.Mask"))
-    (pad "1" thru_hole roundrect (at 0 0) (size 1.7 1.95) (drill 0.95) (layers "*.Cu" "*.Mask") (roundrect_rratio 0.147059)
+    (pad "1" thru_hole roundrect (at 0 0) (size 1.7 1.95) (drill 0.95) (layers "*.Cu" "*.Mask") (roundrect_rratio 0.1470588235)
       (net 4 "GND1") (pinfunction "Pin_1") (pintype "passive"))
     (pad "2" thru_hole oval (at 2.5 0) (size 1.7 1.95) (drill 0.95) (layers "*.Cu" "*.Mask")
@@
     (fp_line (start 4.11 2.7) (end 3.11 2.7)
       (stroke (width 0.1) (type solid)) (layer "F.Fab"))
-    (pad "1" smd roundrect (at -5.04 -2.28 180) (size 2.2 1.2) (layers "F.Cu" "F.Paste" "F.Mask") (roundrect_rratio 0.208333)
+    (pad "1" smd roundrect (at -5.04 -2.28 180) (size 2.2 1.2) (layers "F.Cu" "F.Paste" "F.Mask") (roundrect_rratio 0.2083333333)
       (net 33 "Net-(Q1-G)") (pinfunction "G") (pintype "input"))
-    (pad "2" smd roundrect (at -0.415 -1.525 180) (size 3.05 2.75) (layers "F.Cu" "F.Paste") (roundrect_rratio 0.090909)
+    (pad "2" smd roundrect (at -0.415 -1.525 180) (size 3.05 2.75) (layers "F.Cu" "F.Paste") (roundrect_rratio 0.09090909091)
       (net 20 "Net-(Q1-D)") (pinfunction "D") (pintype "passive"))
-    (pad "2" smd roundrect (at -0.415 1.525 180) (size 3.05 2.75) (layers "F.Cu" "F.Paste") (roundrect_rratio 0.090909)
+    (pad "2" smd roundrect (at -0.415 1.525 180) (size 3.05 2.75) (layers "F.Cu" "F.Paste") (roundrect_rratio 0.09090909091)
       (net 20 "Net-(Q1-D)") (pinfunction "D") (pintype "passive"))
-    (pad "2" smd roundrect (at 1.26 0 180) (size 6.4 5.8) (layers "F.Cu" "F.Mask") (roundrect_rratio 0.043103)
+    (pad "2" smd roundrect (at 1.26 0 180) (size 6.4 5.8) (layers "F.Cu" "F.Mask") (roundrect_rratio 0.04310293103)
       (net 20 "Net-(Q1-D)") (pinfunction "D") (pintype "passive"))
-    (pad "2" smd roundrect (at 2.935 -1.525 180) (size 3.05 2.75) (layers "F.Cu" "F.Paste") (roundrect_rratio 0.090909)
+    (pad "2" smd roundrect (at 2.935 -1.525 180) (size 3.05 2.75) (layers "F.Cu" "F.Paste") (roundrect_rratio 0.09090909091)
       (net 20 "Net-(Q1-D)") (pinfunction "D") (pintype "passive"))
-    (pad "2" smd roundrect (at 2.935 1.525 180) (size 3.05 2.75) (layers "F.Cu" "F.Paste") (roundrect_rratio 0.090909)
+    (pad "2" smd roundrect (at 2.935 1.525 180) (size 3.05 2.75) (layers "F.Cu" "F.Paste") (roundrect_rratio 0.09090909091)
       (net 20 "Net-(Q1-D)") (pinfunction "D") (pintype "passive"))
-    (pad "3" smd roundrect (at -5.04 2.28 180) (size 2.2 1.2) (layers "F.Cu" "F.Paste" "F.Mask") (roundrect_rratio 0.208333)
+    (pad "3" smd roundrect (at -5.04 2.28 180) (size 2.2 1.2) (layers "F.Cu" "F.Paste" "F.Mask") (roundrect_rratio 0.2083333333)
       (net 34 "+12V") (pinfunction "S") (pintype "passive"))
     (model "${KICAD6_3DMODEL_DIR}/Package_TO_SOT_SMD.3dshapes/TO-252-2.wrl"
@@
   )
   (footprint "Capacitor_THT:CP_Radial_D6.3mm_P2.50mm" (layer "F.Cu")
-    (at 77.7 44 90)
+    (at 83.606 59.436)
     (descr "CP, Radial series, Radial, pin pitch=2.50mm, , diameter=6.3mm, Electrolytic Capacitor")
     (tags "CP Radial series Radial pin pitch 2.50mm  diameter 6.3mm Electrolytic Capacitor")
@@
     (zone_connect 2)
     (attr through_hole)
-    (fp_text reference "C1" (at 1.182379 4.2 90) (layer "F.SilkS")
+    (fp_text reference "C1" (at 1.182379 4.2) (layer "F.SilkS")
         (effects (font (size 0.8 0.8) (thickness 0.1)))
     )
-    (fp_text value "100uF" (at 1.25 4.4 90) (layer "F.Fab")
+    (fp_text value "100uF" (at 1.25 4.4) (layer "F.Fab")
         (effects (font (size 0.8 0.8) (thickness 0.1)))
     )
-    (fp_text user "${REFERENCE}" (at 1.25 0 90) (layer "F.Fab")
+    (fp_text user "${REFERENCE}" (at 1.25 0) (layer "F.Fab")
         (effects (font (size 1 1) (thickness 0.15)))
     )
@@
     (fp_circle (center 1.25 0) (end 4.4 0)
       (stroke (width 0.1) (type solid)) (fill none) (layer "F.Fab"))
-    (pad "1" thru_hole rect (at 0 0 90) (size 1.6 1.6) (drill 0.8) (layers "*.Cu" "*.Mask")
-      (net 34 "+12V") (pintype "passive"))
-    (pad "2" thru_hole circle (at 2.5 0 90) (size 1.6 1.6) (drill 0.8) (layers "*.Cu" "*.Mask")
+    (pad "1" thru_hole rect (at 0 0) (size 1.6 1.6) (drill 0.8) (layers "*.Cu" "*.Mask")
+      (net 168 "Logic_Power") (pintype "passive"))
+    (pad "2" thru_hole circle (at 2.5 0) (size 1.6 1.6) (drill 0.8) (layers "*.Cu" "*.Mask")
       (net 1 "GND") (pintype "passive"))
     (model "${KICAD6_3DMODEL_DIR}/Capacitor_THT.3dshapes/CP_Radial_D6.3mm_P2.50mm.wrl"
@@
   (via (at 221.488 135.5344) (size 0.8) (drill 0.4) (layers "F.Cu" "B.Cu") (free) (net 1))
   (via (at 132.7912 42.9006) (size 0.8) (drill 0.4) (layers "F.Cu" "B.Cu") (free) (net 1))
+  (via (at 139.446 25.4) (size 0.8) (drill 0.4) (layers "F.Cu" "B.Cu") (free) (net 1))
   (via (at 187.198 75.946) (size 0.8) (drill 0.4) (layers "F.Cu" "B.Cu") (free) (net 1))
   (via (at 201.676 88.138) (size 0.8) (drill 0.4) (layers "F.Cu" "B.Cu") (free) (net 1))
   (via (at 102.235 68.6562) (size 0.8) (drill 0.4) (layers "F.Cu" "B.Cu") (free) (net 1))
-  (via (at 143.9418 24.8666) (size 0.8) (drill 0.4) (layers "F.Cu" "B.Cu") (free) (net 1))
+  (via (at 144.526 25.146) (size 0.8) (drill 0.4) (layers "F.Cu" "B.Cu") (free) (net 1))
   (via (at 104.648 34.036) (size 0.8) (drill 0.4) (layers "F.Cu" "B.Cu") (free) (net 1))
   (via (at 213.7156 146.1516) (size 0.8) (drill 0.4) (layers "F.Cu" "B.Cu") (free) (net 1))
