File: Circuit/Kicad/V2/RDC_Humanoid_Logic/RDC_Humanoid_Logic.kicad_sch (KiCad schematic)
At the start: 30 parts, among them J1 XT30, J2 Conn_01x03, J3 Conn_01x03, J4 Raspi_connect, Q1 Q_PMOS_GDS, Q2 Q_PMOS_GDS, SW1 SW_SPDT, U4 TBD62783A

Commit message: V2をUpdate。FrontをベタGND、CANトランシーバのSTANDBYとINをGNDに接続、ビアを複数配置、XT30->XT60に更新、D1を回路図通りショットキーバリアダイオードに変更した。
Parts:
- J1: value XT30 -> XT60; footprint Connector_AMASS:AMASS_XT30PW-M_1x02_P2.50mm_Horizontal -> Connector_AMASS:AMASS_XT60PW-M_1x02_P7.20mm_Horizontal
- renumbered C22 to C2, SW1 to SW2, SW1 to SW3
Connections:
- no-connect marks 21 -> 17
Other:
- note added: "STANDBY is Low -> normal mode STANDBY is High -> standby mode (wake up by RXD)"

Commit message: V2基板手直し
Connections:
- no-connect marks 17 -> 46
Changed lines of the file:
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@@
   (junction (at 285.75 229.87) (diameter 0) (color 0 0 0 0)
   )
+  (no_connect (at 269.24 229.87))
   (no_connect (at 104.14 149.86))
   (no_connect (at 104.14 142.24))
+  (no_connect (at 281.94 224.79))
+  (no_connect (at 269.24 227.33))
+  (no_connect (at 281.94 217.17))
   (no_connect (at 205.74 74.93))
+  (no_connect (at 281.94 240.03))
+  (no_connect (at 281.94 214.63))
+  (no_connect (at 281.94 255.27))
   (no_connect (at 124.46 142.24))
   (no_connect (at 104.14 91.44))
+  (no_connect (at 269.24 240.03))
   (no_connect (at 124.46 137.16))
+  (no_connect (at 281.94 245.11))
   (no_connect (at 124.46 149.86))
+  (no_connect (at 269.24 209.55))
+  (no_connect (at 269.24 212.09))
   (no_connect (at 104.14 137.16))
   (no_connect (at 124.46 147.32))
+  (no_connect (at 281.94 250.19))
   (no_connect (at 104.14 139.7))
   (no_connect (at 104.14 144.78))
   (no_connect (at 124.46 144.78))
+  (no_connect (at 269.24 232.41))
+  (no_connect (at 269.24 234.95))
+  (no_connect (at 269.24 224.79))
+  (no_connect (at 281.94 252.73))
+  (no_connect (at 281.94 219.71))
+  (no_connect (at 269.24 207.01))
+  (no_connect (at 281.94 227.33))
+  (no_connect (at 269.24 247.65))
+  (no_connect (at 269.24 245.11))
+  (no_connect (at 281.94 237.49))
+  (no_connect (at 269.24 242.57))
   (no_connect (at 205.74 55.88))
   (no_connect (at 85.09 118.11))
+  (no_connect (at 269.24 252.73))
+  (no_connect (at 281.94 234.95))
+  (no_connect (at 281.94 232.41))
+  (no_connect (at 269.24 250.19))
   (no_connect (at 67.31 127))
+  (no_connect (at 269.24 222.25))
   (no_connect (at 104.14 147.32))
   (no_connect (at 124.46 139.7))
+  (no_connect (at 269.24 219.71))
   (wire (pts (xy 69.85 101.6) (xy 87.63 101.6))
     (stroke (width 0) (type default))

Commit message: 部品表の作成、多少のFootPrint、PCBの変更
Parts:
- D1: footprint Diode_SMD:Vishay_SMPA -> Diode_SMD:D_SOD-123
Changed lines of the file:
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@@
       (effects (font (size 1.27 1.27)) hide)
     )
-    (property "Datasheet" "~" (at 101.6 52.07 0)
+    (property "Datasheet" "https://akizukidenshi.com/goodsaffix/TJ60S04M3L_datasheet_ja_20200624.pdf" (at 101.6 52.07 0)
       (effects (font (size 1.27 1.27)) hide)
     )
@@
       (effects (font (size 1.27 1.27)) hide)
     )
-    (property "Datasheet" "~" (at 101.6 86.36 0)
+    (property "Datasheet" "https://akizukidenshi.com/goodsaffix/2MS1-T1-B4-VS2-Q-E-S.pdf" (at 101.6 86.36 0)
       (effects (font (size 1.27 1.27)) hide)
     )
@@
       (effects (font (size 1.27 1.27)) hide)
     )
-    (property "Datasheet" "~" (at 228.6 209.55 0)
+    (property "Datasheet" "https://www.jst-mfg.com/product/pdf/eng/eXA-WB.pdf?67d6871ee54a2" (at 228.6 209.55 0)
       (effects (font (size 1.27 1.27)) hide)
     )
@@
       (effects (font (size 1.27 1.27)) hide)
     )
-    (property "Datasheet" "~" (at 228.6 248.92 0)
+    (property "Datasheet" "https://www.jst-mfg.com/product/pdf/eng/eXA-WB.pdf?67d6871ee54a2" (at 228.6 248.92 0)
       (effects (font (size 1.27 1.27)) hide)
     )
@@
       (effects (font (size 1.27 1.27)) hide)
     )
-    (property "Datasheet" "~" (at 87.63 113.03 0)
+    (property "Datasheet" "https://akizukidenshi.com/goodsaffix/2MS1-T1-B4-VS2-Q-E-S.pdf" (at 87.63 113.03 0)
       (effects (font (size 1.27 1.27)) hide)
     )
@@
       (effects (font (size 1.27 1.27)) hide)
     )
-    (property "Datasheet" "~" (at 114.3 52.07 0)
+    (property "Datasheet" "https://akizukidenshi.com/goodsaffix/TJ60S04M3L_datasheet_ja_20200624.pdf" (at 114.3 52.07 0)
       (effects (font (size 1.27 1.27)) hide)
     )
@@
       (effects (font (size 1.27 1.27)) hide)
     )
-    (property "Datasheet" "~" (at 69.85 121.92 0)
+    (property "Datasheet" "https://akizukidenshi.com/goodsaffix/2MS1-T1-B4-VS2-Q-E-S.pdf" (at 69.85 121.92 0)
       (effects (font (size 1.27 1.27)) hide)
     )
@@
       (effects (font (size 1.27 1.27)) (justify left))
     )
-    (property "Footprint" "Diode_SMD:Vishay_SMPA" (at 39.37 54.61 0)
+    (property "Footprint" "Diode_SMD:D_SOD-123" (at 39.37 54.61 0)
       (effects (font (size 1.27 1.27)) hide)
     )
@@
       (effects (font (size 1.27 1.27)) hide)
     )
-    (property "Datasheet" "~" (at 55.88 54.61 0)
-      (effects (font (size 1.27 1.27)) hide)
-    )
+    (property "Datasheet" "https://akizukidenshi.com/catalog/g/g102724/" (at 55.88 54.61 0)
+      (effects (font (size 1.27 1.27)) hide)
+    )

Commit message: gbrの生成
Connections:
- net +12V: no longer C1.1
- net Logic_Power: now also C1.1
Other:
- moved on the sheet: C1
Changed lines of the file:
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@@
   (junction (at 39.37 49.53) (diameter 0) (color 0 0 0 0)
   )
+  (junction (at 124.46 49.53) (diameter 0) (color 0 0 0 0)
+  )
   (junction (at 92.71 49.53) (diameter 0) (color 0 0 0 0)
   )
@@
   )
   (junction (at 101.6 60.96) (diameter 0) (color 0 0 0 0)
-  )
-  (junction (at 55.88 49.53) (diameter 0) (color 0 0 0 0)
   )
   (junction (at 285.75 229.87) (diameter 0) (color 0 0 0 0)
@@
     (stroke (width 0) (type default))
   )
-  (wire (pts (xy 60.96 49.53) (xy 55.88 49.53))
+  (wire (pts (xy 39.37 49.53) (xy 60.96 49.53))
     (stroke (width 0) (type default))
   )
@@
     (stroke (width 0) (type default))
   )
+  (wire (pts (xy 109.22 49.53) (xy 106.68 49.53))
+    (stroke (width 0) (type default))
+  )
   (wire (pts (xy 87.63 101.6) (xy 87.63 107.95))
     (stroke (width 0) (type default))
@@
     (stroke (width 0) (type default))
   )
-  (wire (pts (xy 55.88 49.53) (xy 55.88 52.07))
-    (stroke (width 0) (type default))
-  )
-  (wire (pts (xy 55.88 58.42) (xy 55.88 57.15))
+  (wire (pts (xy 124.46 49.53) (xy 124.46 52.07))
+    (stroke (width 0) (type default))
+  )
+  (wire (pts (xy 124.46 58.42) (xy 124.46 57.15))
     (stroke (width 0) (type default))
   )
@@
     (stroke (width 0) (type default))
   )
+  (wire (pts (xy 124.46 49.53) (xy 130.81 49.53))
+    (stroke (width 0) (type default))
+  )
   (wire (pts (xy 83.82 49.53) (xy 83.82 52.07))
     (stroke (width 0) (type default))
@@
     (stroke (width 0) (type default))
   )
-  (wire (pts (xy 39.37 49.53) (xy 55.88 49.53))
-    (stroke (width 0) (type default))
-  )
   (wire (pts (xy 101.6 210.82) (xy 107.95 210.82))
     (stroke (width 0) (type default))
@@
     (stroke (width 0) (type default))
   )
-  (wire (pts (xy 119.38 49.53) (xy 130.81 49.53))
-    (stroke (width 0) (type default))
-  )
   (wire (pts (xy 83.82 60.96) (xy 92.71 60.96))
     (stroke (width 0) (type default))
   )
-  (wire (pts (xy 106.68 49.53) (xy 109.22 49.53))
-    (stroke (width 0) (type default))
-  )
   (wire (pts (xy 130.81 101.6) (xy 130.81 49.53))
     (stroke (width 0) (type default))
@@
   )
   (wire (pts (xy 281.94 222.25) (xy 285.75 222.25))
+    (stroke (width 0) (type default))
+  )
+  (wire (pts (xy 124.46 49.53) (xy 119.38 49.53))
     (stroke (width 0) (type default))
   )
@@
     )
   )
-  (symbol (lib_id "power:GND") (at 55.88 58.42 0) (unit 1)
-    (in_bom yes) (on_board yes) (dnp no) (fields_autoplaced)
-    (property "Reference" "#PWR04" (at 55.88 64.77 0)
-      (effects (font (size 1.27 1.27)) hide)
-    )
-    (property "Value" "GND" (at 55.88 63.5 0)
-      (effects (font (size 1.27 1.27)))
-    )
-    (property "Footprint" "" (at 55.88 58.42 0)
-      (effects (font (size 1.27 1.27)) hide)
-    )
-    (property "Datasheet" "" (at 55.88 58.42 0)
+  (symbol (lib_id "power:GND") (at 124.46 58.42 0) (unit 1)
+    (in_bom yes) (on_board yes) (dnp no) (fields_autoplaced)
+    (property "Reference" "#PWR04" (at 124.46 64.77 0)
+      (effects (font (size 1.27 1.27)) hide)
+    )
+    (property "Value" "GND" (at 124.46 63.5 0)
+      (effects (font (size 1.27 1.27)))
+    )
+    (property "Footprint" "" (at 124.46 58.42 0)
+      (effects (font (size 1.27 1.27)) hide)
+    )
+    (property "Datasheet" "" (at 124.46 58.42 0)
       (effects (font (size 1.27 1.27)) hide)
     )
@@
     )
   )
-  (symbol (lib_id "Device:C_Polarized_Small") (at 55.88 54.61 0) (unit 1)
-    (in_bom yes) (on_board yes) (dnp no) (fields_autoplaced)
-    (property "Reference" "C1" (at 58.42 52.7939 0)
-      (effects (font (size 1.27 1.27)) (justify left))
-    )
-    (property "Value" "100uF" (at 58.42 55.3339 0)
-      (effects (font (size 1.27 1.27)) (justify left))
-    )
-    (property "Footprint" "Capacitor_THT:CP_Radial_D6.3mm_P2.50mm" (at 55.88 54.61 0)
-      (effects (font (size 1.27 1.27)) hide)
-    )
-    (property "Datasheet" "https://akizukidenshi.com/catalog/g/g102724/" (at 55.88 54.61 0)
-      (effects (font (size 1.27 1.27)) hide)
-    )
+  (symbol (lib_id "Device:C_Polarized_Small") (at 124.46 54.61 0) (unit 1)
+    (in_bom yes) (on_board yes) (dnp no) (fields_autoplaced)
+    (property "Reference" "C1" (at 127 52.7939 0)
+      (effects (font (size 1.27 1.27)) (justify left))
+    )
+    (property "Value" "100uF" (at 127 55.3339 0)
+      (effects (font (size 1.27 1.27)) (justify left))
+    )
+    (property "Footprint" "Capacitor_THT:CP_Radial_D6.3mm_P2.50mm" (at 124.46 54.61 0)
+      (effects (font (size 1.27 1.27)) hide)
+    )
+    (property "Datasheet" "https://akizukidenshi.com/catalog/g/g102724/" (at 124.46 54.61 0)
+      (effects (font (size 1.27 1.27)) hide)
+    )
