Commit message: 脛と足を別パーツ化

File: Robot_Models/URDF/urdf_simple-model/simple_model.urdf (robot description, URDF)
Before this commit: robot rdc_biped_robot, 8 links, 7 joints
Links:
- added link None, mass 0.0; collision mesh filename=meshes/stl/link_heel2end.stl scale=1 1 1; visual mesh filename=meshes/stl/link_heel2end.stl scale=1 1 1
- link body: mass 0.1 -> 1.782
- link l_kp2heel: mass 0.1 -> 1
- link l_wp2kp: mass 0.1 -> 1
- link l_wr2wp: mass 0.1 -> 1.782
- link r_kp2heel: mass 0.1 -> 1
- link r_wp2kp: mass 0.1 -> 1
- link r_wr2wp: mass 0.1 -> 1.782
Joints:
- added joint l_ankle: type fixed, parent l_kp2heel, child l_heel2end, origin xyz=-0.164 rpy=0 0 0
- added joint r_ankle: type fixed, parent r_kp2heel, child r_heel2end, origin xyz=-0.164 rpy=0 0 0
- joint l_knee_pitch: limit lower=-1.72 upper=1.72 effort=100 velocity=100 -> lower=-6.28 upper=6.28 effort=7.2 velocity=11.519173063
- joint l_waist_pitch: limit lower=-1.72 upper=1.72 effort=100 velocity=100 -> lower=-6.28 upper=6.28 effort=7.2 velocity=11.519173063
- joint l_waist_roll: limit lower=-1.72 upper=1.72 effort=100 velocity=100 -> lower=-6.28 upper=6.28 effort=7.2 velocity=11.519173063; origin xyz=0 0.105 0 rpy=0 0 0 -> xyz=0 0.105 0.364 rpy=0 0 0
- joint r_knee_pitch: limit lower=-1.72 upper=1.72 effort=100 velocity=100 -> lower=-6.28 upper=6.28 effort=7.2 velocity=11.519173063
- joint r_waist_pitch: limit lower=-1.72 upper=1.72 effort=100 velocity=100 -> lower=-6.28 upper=6.28 effort=7.2 velocity=11.519173063
- joint r_waist_roll: limit lower=-1.72 upper=1.72 effort=100 velocity=100 -> lower=-6.28 upper=6.28 effort=7.2 velocity=11.519173063; origin xyz=0 -0.105 0 rpy=0 0 0 -> xyz=0 -0.105 0.364 rpy=0 0 0

Commit message: simple_modelに胴体を搭載。寸法・質量・慣性をUpdate。それっぽい感じになったのでよし。

File: Robot_Models/URDF/urdf_simple-model/simple_model.urdf (robot description, URDF)
Before this commit: robot rdc_biped_robot, 9 links, 9 joints
Links:
- removed link None
- added link body_luggage, mass 6.002284; collision mesh filename=meshes/stl/body_luggage.stl scale=1 1 1; visual mesh filename=meshes/stl/body_luggage.stl scale=1 1 1
- added link l_heel2end, mass 0.0; collision mesh filename=meshes/stl/link_heel2end.stl scale=1 1 1; visual mesh filename=meshes/stl/link_heel2end.stl scale=1 1 1
- added link r_heel2end, mass 0.0; collision mesh filename=meshes/stl/link_heel2end.stl scale=1 1 1; visual mesh filename=meshes/stl/link_heel2end.stl scale=1 1 1
- link body: mass 1.782 -> 1.128279
- link l_kp2heel: mass 1 -> 0.199496
- link l_wp2kp: mass 1 -> 0.581098
- link l_wr2wp: mass 1.782 -> 1.463019
- link r_kp2heel: mass 1 -> 0.199496
- link r_wp2kp: mass 1 -> 0.581098
- link r_wr2wp: mass 1.782 -> 1.463019
Joints:
- removed joint base_joint
- added joint CPG: type fixed, parent base_link, child body, origin xyz=0 0 0.333 rpy=0 0 0
- added joint luggage: type fixed, parent body, child body_luggage, origin xyz=-0.091 0 0 rpy=0 0 0
- joint l_ankle: origin xyz=-0.164 rpy=0 0 0 -> xyz=0 0 -0.149335 rpy=0 0 0
- joint l_knee_pitch: origin xyz=0 0 -0.18 rpy=0 0 0 -> xyz=0 0 -0.16 rpy=0 0 0
- joint l_waist_pitch: origin xyz=0.08 0.041 0.00 rpy=0 0 0 -> xyz=0.091 0.055 0.00 rpy=0 0 0
- joint l_waist_roll: origin xyz=0 0.105 0.364 rpy=0 0 0 -> xyz=-0.091 0.075 0 rpy=0 0 0
- joint r_ankle: origin xyz=-0.164 rpy=0 0 0 -> xyz=0 0 -0.149335 rpy=0 0 0
- joint r_knee_pitch: origin xyz=0 0 -0.18 rpy=0 0 0 -> xyz=0 0 -0.16 rpy=0 0 0
- joint r_waist_pitch: origin xyz=0.08 -0.041 0.00 rpy=0 0 0 -> xyz=0.091 -0.055 0.00 rpy=0 0 0
- joint r_waist_roll: origin xyz=0 -0.105 0.364 rpy=0 0 0 -> xyz=-0.091 -0.075 0 rpy=0 0 0
