File: Circuit/Kicad/V2/RDC_Humanoid_Power_Kicad9/RDC_Humanoid_Power.kicad_sch (KiCad schematic)
At the start: 10 parts, among them J1 LiPo_+24V, J2 LiPo_+24V, J3 SteadyWin_8108, J4 SteadyWin_8108, J5 SteadyWin_8108, J6 SteadyWin_8108, J7 SteadyWin_8108, J8 SteadyWin_8108, K1 Relay_SPST-NO

Commit message: power側の回路をUpdate
Parts:
- added J10, J9: XT60, symbol Connector_Generic:Conn_02x02_Row_Letter_Last
- D1: value D -> VS-VSKD166/16PBF
- K1: value Relay_SPST-NO -> G9EC-1-B-DC12
Connections:
- net +48V: now also J9.1b (Pin_1b); no longer J1.1 (Pin_1)
- net GND: now also J10.2b (Pin_2b); no longer J2.2 (Pin_2)
- net at J1.2 (Pin_2): now also J9.2a (Pin_2a); no longer J2.1 (Pin_1)
- new net: J1.1 (Pin_1), J9.1a (Pin_1a)
- new net: J10.1a (Pin_1a), J2.1 (Pin_1)
- new net: J10.2a (Pin_2a), J2.2 (Pin_2)
- new net: J10.1b (Pin_1b), J9.2b (Pin_2b)
Other:
- note added: "CANチェーン用基板"
- note added: "端子台"
- note removed: "ギボシ端子"
- note removed: "ギボシ端子ダブル"
- moved on the sheet: J1, J2
