File: Circuit/Kicad/V3/RDC_Humanoid_Logic/RDC_Humanoid_Logic.kicad_sch (KiCad schematic)
At the start: 29 parts, among them J1 XT60, J2 Conn_01x03, J3 Conn_01x03, J4 Raspi_connect, Q1 Q_PMOS_GDS, Q2 Q_PMOS_GDS, SW1 SW_SPDT, SW2 SW_SPDT, SW3 SW_SPDT, U4 TBD62085AFWG

Commit message: logic V3のトランジスタアレイ周りを修正
Parts:
- added J5: 74AHC1G04W5, Package_TO_SOT_SMD:SOT-23-5, symbol Connector_Generic:Conn_02x03_Counter_Clockwise
- J4: pin header (none) -> https://www.raspberrypi.com/documentation/computers/raspber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
- SW2: val (none) -> STM
- SW3: val (none) -> RPI5
- U4: value TBD62085AFWG -> TBD62083AFG
Connections:
- net EN_Power: now also U4.10 (COMMON)
- net EN_STM: now also J5.2 (Pin_2)
- net GND: now also J5.3 (Pin_3)
- net Logic_Power/EN_RasPi_Power: now also U4.11 (O8)
- net Logic_Power/EN_STM_Power: now also U4.12 (O7)
- net EN_STM_VCC: now reaches J4.1 (Pin_1)
- net EN_STM_VCC: now also J5.5 (Pin_5)
- net at SW3.1 (A): now also R8.1, U4.8 (I8)
- net at SW3.3 (C): no longer R8.1
- net at R7.1: now also SW2.1 (A), U4.7 (I7), J5.4 (Pin_4); no longer SW2.3 (C)
Other:
- note added: "3V3"
- note added: "B接点"
- note added: "修正済み"
- moved on the sheet: R7, U4
